Commit message: add lourakis lm

File: src/its/urdf/fingertip.urdf.xacro (robot description, xacro)
@@ -2,5 +2,5 @@
 <robot xmlns:xacro="http://www.ros.org/wiki/xacro" name="fingertip">
   <!-- Fingertip -->
-  <link name="TacTip"/>
+  <link name="DigiTac"/>
   <joint name="fingertip_to_brush" type="fixed">
       <parent link="panda_link8"/>
